Commit message: test deployment

File: src/jetracer_description/urdf/jetracer.urdf.xacro (robot description, xacro)
@@ -199,4 +199,14 @@
     <origin xyz="${camera_x} ${camera_y} ${camera_z}" rpy="0 0 0"/>
   </joint>
+  <!-- Camera optical frame: standard ROS convention for CSI cameras -->
+  <link name="camera_link_optical">
+    <xacro:box_inertia mass="0.0001" x="0.001" y="0.001" z="0.001"/>
+  </link>
+  <joint name="camera_optical_joint" type="fixed">
+    <parent link="camera_link"/>
+    <child link="camera_link_optical"/>
+    <!-- Rotate to align with optical axis (Z forward, X right, Y down) -->
+    <origin xyz="0 0 0" rpy="${-pi/2} 0 ${-pi/2}"/>
+  </joint>
   <link name="imu_link">
     <visual>

Commit message: update

File: src/jetracer_description/urdf/jetracer.urdf.xacro (robot description, xacro)
@@ -1,5 +1,5 @@
 <?xml version="1.0"?>
 <robot name="jetracer" xmlns:xacro="http://www.ros.org/wiki/xacro">
-  <xacro:property name="pi" value="3.1415926535897931"/>
+  <xacro:property name="half_pi" value="${xacro.pi / 2.0}"/>
   <xacro:property name="wheelbase" value="0.255"/>
   <xacro:property name="track_width" value="0.180"/>
